Commit message: same issue for collision

File: abc.urdf (robot description, URDF)
Before this commit: robot abc, 3 links, 2 joints
Links:
- link a_link: geometry collision mesh filename=package://rviz_melodic_urdf_issue/a.dae scale=1.0 1.0 1.0; visual mesh filename=package://rviz_melodic_urdf_issue/a.dae scale=1.0 1.0 1.0
- link b_link: geometry collision mesh filename=package://rviz_melodic_urdf_issue/b.dae scale=1.0 1.0 1.0; visual mesh filename=package://rviz_melodic_urdf_issue/b.dae scale=1.0 1.0 1.0
- link c_link: geometry collision mesh filename=package://rviz_melodic_urdf_issue/c.dae scale=1.0 1.0 1.0; visual mesh filename=package://rviz_melodic_urdf_issue/c.dae scale=1.0 1.0 1.0
